File: 0.81OLED_DevBoard_Hardware/0.87OLED_DevBoard.kicad_sch (KiCad schematic)
At the start: 15 parts, among them IC1 XC6206P332MR, J1 Connector_Pin, U1 中景园_0.87寸OLED

Commit message: Finish PCB Layout
Parts:
- C1, C2, C3, C4, C5, C6, C7, C8: symbol Device:C -> oled:C
- IC1: symbol SamacSys_Parts:XC6206P332MR -> oled:XC6206P332MR
- J1: symbol Connector:Conn_01x04_Pin -> oled:Conn_01x04_Pin
- R1, R2, R3, R4: symbol Device:R -> oled:R
- U1: symbol kicad_lceda:中景园_0.87寸OLED -> oled:中景园_0.87寸OLED
Changed lines of the file:
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@@
     (effects (font (size 1.27 1.27)) (justify left bottom))
   )
-  (symbol (lib_id "Device:C") (at 114.3 107.442 90) (unit 1)
+  (symbol (lib_id "oled:C") (at 114.3 107.442 90) (unit 1)
     (in_bom yes) (on_board yes) (dnp no)
     (property "Reference" "C6" (at 112.014 106.426 90)
@@
     )
   )
-  (symbol (lib_id "Device:R") (at 70.104 117.348 0) (unit 1)
+  (symbol (lib_id "oled:R") (at 70.104 117.348 0) (unit 1)
     (in_bom yes) (on_board yes) (dnp no)
     (property "Reference" "R4" (at 70.104 118.618 90)
@@
     )
   )
-  (symbol (lib_id "Device:C") (at 117.348 80.772 90) (unit 1)
+  (symbol (lib_id "oled:C") (at 117.348 80.772 90) (unit 1)
     (in_bom yes) (on_board yes) (dnp no)
     (property "Reference" "C2" (at 115.062 79.756 90)
@@
     )
   )
-  (symbol (lib_id "Device:C") (at 114.3 112.522 90) (unit 1)
+  (symbol (lib_id "oled:C") (at 114.3 112.522 90) (unit 1)
     (in_bom yes) (on_board yes) (dnp no)
     (property "Reference" "C7" (at 112.014 111.506 90)
@@
     )
   )
-  (symbol (lib_id "Connector:Conn_01x04_Pin") (at 36.83 63.754 0) (unit 1)
+  (symbol (lib_id "oled:Conn_01x04_Pin") (at 36.83 63.754 0) (unit 1)
     (in_bom yes) (on_board yes) (dnp no) (fields_autoplaced)
     (property "Reference" "J1" (at 37.465 55.88 0)
@@
     )
   )
-  (symbol (lib_id "Device:C") (at 114.3 117.602 90) (unit 1)
+  (symbol (lib_id "oled:C") (at 114.3 117.602 90) (unit 1)
     (in_bom yes) (on_board yes) (dnp no)
     (property "Reference" "C8" (at 112.014 116.586 90)
@@
     )
   )
-  (symbol (lib_id "Device:C") (at 117.348 75.692 90) (unit 1)
+  (symbol (lib_id "oled:C") (at 117.348 75.692 90) (unit 1)
     (in_bom yes) (on_board yes) (dnp no)
     (property "Reference" "C1" (at 115.062 74.676 90)
@@
     )
   )
-  (symbol (lib_id "Device:C") (at 86.868 101.092 180) (unit 1)
+  (symbol (lib_id "oled:C") (at 86.868 101.092 180) (unit 1)
     (in_bom yes) (on_board yes) (dnp no)
     (property "Reference" "C5" (at 88.392 99.06 0)
@@
     )
   )
-  (symbol (lib_id "Device:R") (at 86.868 90.932 0) (unit 1)
+  (symbol (lib_id "oled:R") (at 86.868 90.932 0) (unit 1)
     (in_bom yes) (on_board yes) (dnp no)
     (property "Reference" "R1" (at 86.868 92.202 90)
@@
     )
   )
-  (symbol (lib_id "Device:C") (at 104.14 88.646 90) (unit 1)
+  (symbol (lib_id "oled:C") (at 104.14 88.646 90) (unit 1)
     (in_bom yes) (on_board yes) (dnp no)
     (property "Reference" "C4" (at 101.854 87.63 90)
@@
     )
   )
-  (symbol (lib_id "Device:C") (at 104.14 93.472 90) (unit 1)
+  (symbol (lib_id "oled:C") (at 104.14 93.472 90) (unit 1)
     (in_bom yes) (on_board yes) (dnp no)
     (property "Reference" "C3" (at 101.854 92.456 90)
@@
     )
   )
-  (symbol (lib_id "Device:R") (at 114.554 103.632 90) (unit 1)
+  (symbol (lib_id "oled:R") (at 114.554 103.632 90) (unit 1)
     (in_bom yes) (on_board yes) (dnp no)
     (property "Reference" "R2" (at 115.824 103.632 90)
@@
     )
   )
-  (symbol (lib_id "SamacSys_Parts:XC6206P332MR") (at 111.76 56.896 0) (mirror y) (unit 1)
+  (symbol (lib_id "oled:XC6206P332MR") (at 111.76 56.896 0) (mirror y) (unit 1)
     (in_bom yes) (on_board yes) (dnp no)
     (property "Reference" "IC1" (at 97.79 49.022 0)
@@
     )
   )
-  (symbol (lib_id "kicad_lceda:中景园_0.87寸OLED") (at 128.016 90.932 0) (unit 1)
+  (symbol (lib_id "oled:中景园_0.87寸OLED") (at 128.016 90.932 0) (unit 1)
     (in_bom yes) (on_board yes) (dnp no) (fields_autoplaced)
     (property "Reference" "U1" (at 138.938 90.932 0)
@@
     )
   )
-  (symbol (lib_id "Device:R") (at 65.786 117.348 0) (unit 1)
+  (symbol (lib_id "oled:R") (at 65.786 117.348 0) (unit 1)
     (in_bom yes) (on_board yes) (dnp no)
     (property "Reference" "R3" (at 65.786 118.618 90)
